File: Hardware/MicroMod-Big Display-Carrier.brd (EAGLE design)
At the start: 58.4 x 45.7 mm, 121 parts, among them J11 microSD, J2 JTAG, J3 Qwiic, J4 MICROMOD-2222-C, J5 SPI, J6 UART, J7 HDMI, J8 Dedicated, U5 AP7361C-33FGE

Commit message: Update silk
Parts:
- U$3, U$5: device output:DISPLAY0 -> output:BIG_DISPLAY0
- moved U$24 13.0 mm to (25.4, 33.0)
- moved U$3 11.1 mm to (36.8, 33.0)
- moved U$5 0.25 mm to (29.1, 19.6)
Changed lines of the file:
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@@
 <layer number="47" name="Measures" color="7" fill="1" visible="no" active="yes"/>
 <layer number="48" name="Document" color="7" fill="1" visible="no" active="yes"/>
-<layer number="49" name="Reference" color="7" fill="1" visible="yes" active="yes"/>
+<layer number="49" name="Reference" color="7" fill="1" visible="no" active="yes"/>
 <layer number="50" name="dxf" color="7" fill="1" visible="no" active="yes"/>
 <layer number="51" name="tDocu" color="6" fill="1" visible="yes" active="yes"/>
@@
 <attribute name="VALUE" x="23.495" y="20.32" size="0.762" layer="27" rot="R270" align="center"/>
 </element>
-<element name="U$24" library="SparkFun-MicroMod" package="MICROMOD_LOGO_.35" value="" x="38.354" y="32.766" smashed="yes"/>
+<element name="U$24" library="SparkFun-MicroMod" package="MICROMOD_LOGO_.35" value="" x="25.4" y="33.02" smashed="yes"/>
 <element name="J9" library="SparkFun-Connectors" package="1X01_NO_SILK" value="" x="17.78" y="3.81" smashed="yes">
 <attribute name="NAME" x="16.51" y="4.953" size="0.6096" layer="25" font="vector" ratio="20"/>
@@
 </element>
 <element name="U$2" library="output" package="MICROSD0" value="" x="10.033" y="24.384" smashed="yes"/>
-<element name="U$3" library="output" package="DISPLAY0" value="" x="47.879" y="32.766" smashed="yes"/>
-<element name="U$5" library="output" package="DISPLAY0" value="" x="29.083" y="19.304" smashed="yes" rot="MR0"/>
 <element name="U$1" library="SparkX" package="SPARKX-MEDIUM" value="SPARKX-LOGO4" x="44.45" y="35.56" smashed="yes"/>
 <element name="U$22" library="SparkX" package="SPARKX-MEDIUM" value="SPARKX-LOGO4" x="29.21" y="24.13" smashed="yes" rot="MR0"/>
+<element name="U$3" library="output" package="BIG_DISPLAY0" value="" x="36.83" y="33.02" smashed="yes"/>
+<element name="U$5" library="output" package="BIG_DISPLAY0" value="" x="29.083" y="19.558" smashed="yes" rot="MR0"/>
 </elements>
 <signals>
