File: Hardware/Production/MicroMod-Big Display-Carrier-Panel.brd (EAGLE design)
At the start: 146.6 x 151.9 mm, 726 parts, among them J11 microSD, J13 Qwiic, J15 JTAG, J16 SPI, J17 Dedicated, J19 microSD, J2 JTAG, J20 UART, J22 MICROMOD-2222-C, J24 HDMI, J26 Qwiic, J27 JTAG, J28 SPI, J29 Dedicated, J3 Qwiic, J31 microSD, J32 UART, J34 MICROMOD-2222-C, J36 HDMI, J38 Qwiic, J39 JTAG, J4 MICROMOD-2222-C, J40 SPI, J41 Dedicated, J43 microSD, J44 UART, J46 MICROMOD-2222-C, J48 HDMI, J5 SPI, J50 Qwiic, J51 JTAG, J52 SPI, J53 Dedicated, J55 microSD, J56 UART, J58 MICROMOD-2222-C, J6 UART, J60 HDMI, J62 Qwiic, J63 JTAG, J64 SPI, J65 Dedicated, J67 microSD, J68 UART, J7 HDMI, J70 MICROMOD-2222-C, J72 HDMI, J8 Dedicated, U1 AP7361C-33FGE, U2 AP7361C-33FGE, U3 AP7361C-33FGE, U4 AP7361C-33FGE, U5 AP7361C-33FGE, U6 AP7361C-33FGE

Commit message: Update silk
Parts:
- U$113, U$114, U$171, U$172, U$229, U$230, U$287, U$288, U$345, U$346: value (none) -> SPARKX-LOGO4; device output:DISPLAY0 -> SparkX:SPARKX-MEDIUM
- U$115, U$116, U$173, U$174, U$231, U$232, U$289, U$290, U$347, U$348: value SPARKX-LOGO4 -> (none); device SparkX:SPARKX-MEDIUM -> output:BIG_DISPLAY0
- U$3, U$5: device output:DISPLAY0 -> output:BIG_DISPLAY0
- moved U$117 13.0 mm to (25.4, 79.2)
- moved U$233 13.0 mm to (25.4, 125.5)
- moved U$24 13.0 mm to (25.4, 33.0)
- moved U$175 13.0 mm to (87.4, 79.2)
- moved U$26 13.0 mm to (87.4, 33.0)
- moved U$291 13.0 mm to (87.4, 125.5)
- moved U$3 11.1 mm to (36.8, 33.0)
- moved U$115 8.03 mm to (98.8, 33.0)
- moved U$173 8.03 mm to (36.8, 79.2)
- moved U$231 8.03 mm to (98.8, 79.2)
- moved U$289 8.03 mm to (36.8, 125.5)
- moved U$347 8.03 mm to (98.8, 125.5)
- moved U$172 4.83 mm to (29.2, 70.4)
- moved U$230 4.83 mm to (91.2, 70.4)
- moved U$114 4.83 mm to (91.2, 24.1)
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